Commit message: Gazebo上に綿あめ器つくるlaunchファイル作ったよ

File: urdf/CandyFlossMaker.urdf (robot description, URDF)
Before this commit: robot CandyFlossMaker, 2 links, 1 joints
Links:
- link base_link: geometry collision mesh filename=package://candy_floss/meshes/CandyFlossMaker.stl; visual mesh filename=package://candy_floss/meshes/CandyFlossMaker.stl scale=0.001 0.001 0.001
